Commit message: wip

File: urdf/base_omni.xacro (robot description, xacro)
@@ -7,4 +7,7 @@
   <xacro:property name="base_z_size" value="0.20" />
   <xacro:macro name="omnibase" params="prefix *origin">
+    <material name="dark_cyan">
+      <color rgba="0 0.55 0.55 1.0"/>
+    </material>
     <!-- Base footprint is on the ground under the robot -->
     <link name="${prefix}base_footprint">
@@ -69,4 +72,5 @@
           <cylinder length="0.05" radius="0.1"/>
         </geometry>
+        <material name="dark_cyan"/>
       </visual>
       <collision>
@@ -85,4 +89,5 @@
           <cylinder length="0.05" radius="0.1"/>
         </geometry>
+        <material name="dark_cyan"/>
       </visual>
       <collision>
@@ -101,4 +106,5 @@
           <cylinder length="0.05" radius="0.1"/>
         </geometry>
+        <material name="dark_cyan"/>
       </visual>
       <collision>
@@ -117,4 +123,5 @@
           <cylinder length="0.05" radius="0.1"/>
         </geometry>
+        <material name="dark_cyan"/>
       </visual>
       <collision>
